File: kudox/pcb/kicad_files/kudox.kicad_pcb (KiCad board)
At the start: 2 copper layers, 162.2 x 126.5 mm, 86 parts, among them K0 KEYSW, K1 KEYSW, K10 KEYSW, K11 KEYSW, K12 KEYSW, K13 KEYSW, K14 KEYSW, K15 KEYSW, K16 KEYSW, K2 KEYSW, K20 KEYSW, K21 KEYSW, K22 KEYSW, K23 KEYSW, K24 KEYSW, K25 KEYSW, K26 KEYSW, K3 KEYSW, K30 KEYSW, K31 KEYSW, K32 KEYSW, K33 KEYSW, K34 KEYSW, K35 KEYSW, K36 KEYSW, K4 KEYSW, K40 KEYSW, K41 KEYSW, K42 KEYSW, K43 KEYSW, K44 KEYSW, K45 KEYSW, K46 KEYSW, K5 KEYSW, K6 KEYSW, U1 ProMicro

Commit message: Modified pcb.
Parts:
- removed D26, D36, D6: D, Keebio-Parts:Diode-dual
- removed K26, K36, K6: KEYSW, canadian_footprints:Mx_Alps_100-dualside
- added HOLE_M3: VAL**, keyboard_parts:HOLE_M3, F.Cu at (181.5, 157.9)
- moved RST_SW1 125.6 mm to (209.5, 133.7)
- moved U1 53.4 mm to (202.7, 80.0), turned to 180 degrees
- moved RGB_STRIP1 51.5 mm to (230.8, 61.2)
- moved R1 31.0 mm to (211.2, 30.3)
- moved R2 31.0 mm to (225.4, 30.3)
- moved TRRS1 31.0 mm to (218.3, 21.6)
- moved HOLE_M3 30.1 mm to (83.2, 106.1)
- moved D16 27.2 mm to (202.5, 80.0), turned to 90 degrees
- moved HOLE_M3 26.3 mm to (105.0, 71.9)
- moved D31 22.4 mm to (134.7, 126.4)
- moved K31 22.4 mm to (134.7, 118.2)
- moved D35 22.0 mm to (211.0, 126.4)
- moved K35 22.0 mm to (211.0, 118.1)
- moved D32 21.8 mm to (153.9, 126.4)
- moved K32 21.8 mm to (153.9, 118.1)
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Routing:
- net col1: track 144.0 -> 265.6 mm
- net col0: track 167.6 -> 257.1 mm
- net rgb_data: track 103.7 -> 18.4 mm, vias 2 -> 0
- net col6: track 184.3 -> 101.4 mm
- net row4: track 189.3 -> 232.7 mm, vias 0 -> 2
- net col2: track 119.8 -> 160.5 mm, vias 0 -> 2
- net RST: track 47.1 -> 9.88 mm
- net col3: track 97.8 -> 120.4 mm
- net col4: track 103.1 -> 124.4 mm
- net SCL: track 80.1 -> 59.4 mm, vias 2 -> 0
- net SDA: track 71.4 -> 52.9 mm
- net row3: track 207.9 -> 189.5 mm, vias 1 -> 2
- net Net-(D26-Pad2): track 15.6 -> 0.00 mm
- net row1: track 169.3 -> 154.0 mm, vias 1 -> 0
- net Net-(D36-Pad2): track 15.1 -> 0.00 mm
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- removed copper zone on B.Cu, net GND
- removed copper zone on F.Cu, net GND
Other:
- board size 162.2 x 126.5 mm -> 143.6 x 129.5 mm
