File: kudox/pcb/kicad_files/kudox.sch (KiCad schematic (older format))
At the start: 76 parts, among them K0 KEYSW, K1 KEYSW, K10 KEYSW, K11 KEYSW, K12 KEYSW, K13 KEYSW, K14 KEYSW, K15 KEYSW, K16 KEYSW, K2 KEYSW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

Commit message: Modified pcb.
Parts:
- removed D26, D36, D6: D, Keebio-Parts:Diode-dual, symbol D
- removed K26, K36, K6: KEYSW, Keebio-Parts:Hybrid_PCB_100H_Dual_hole-nosilk, symbol KEYSW
